File: multisonar.sch (EAGLE design)
At the start: 0 parts

Commit message: Add ultrasonic sensors
Parts:
- added J_ULTRASONIC_1, J_ULTRASONIC_2, J_ULTRASONIC_3, J_ULTRASONIC_4, J_ULTRASONIC_5, J_ULTRASONIC_6, J_ULTRASONIC_7, J_ULTRASONIC_8: HC-SR04, Ultrasonic Sensor HC-SR04:HC-SR04
Changed lines of the file:
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@@
 <setting verticaltext="up"/>
 </settings>
-<grid distance="0.1" unitdist="inch" unit="inch" style="lines" multiple="1" display="no" altdistance="0.01" altunitdist="inch" altunit="inch"/>
+<grid distance="0.1" unitdist="inch" unit="inch" style="lines" multiple="1" display="yes" altdistance="0.01" altunitdist="inch" altunit="inch"/>
 <layers>
+<layer number="1" name="Top" color="4" fill="1" visible="no" active="no"/>
+<layer number="16" name="Bottom" color="1" fill="1" visible="no" active="no"/>
+<layer number="17" name="Pads" color="2" fill="1" visible="no" active="no"/>
+<layer number="18" name="Vias" color="2" fill="1" visible="no" active="no"/>
+<layer number="19" name="Unrouted" color="6" fill="1" visible="no" active="no"/>
+<layer number="20" name="Dimension" color="15" fill="1" visible="no" active="no"/>
+<layer number="21" name="tPlace" color="7" fill="1" visible="no" active="no"/>
+<layer number="22" name="bPlace" color="7" fill="1" visible="no" active="no"/>
+<layer number="23" name="tOrigins" color="15" fill="1" visible="no" active="no"/>
+<layer number="24" name="bOrigins" color="15" fill="1" visible="no" active="no"/>
+<layer number="25" name="tNames" color="7" fill="1" visible="no" active="no"/>
+<layer number="26" name="bNames" color="7" fill="1" visible="no" active="no"/>
+<layer number="27" name="tValues" color="7" fill="1" visible="no" active="no"/>
+<layer number="28" name="bValues" color="7" fill="1" visible="no" active="no"/>
+<layer number="29" name="tStop" color="7" fill="3" visible="no" active="no"/>
+<layer number="30" name="bStop" color="7" fill="6" visible="no" active="no"/>
+<layer number="31" name="tCream" color="7" fill="4" visible="no" active="no"/>
+<layer number="32" name="bCream" color="7" fill="5" visible="no" active="no"/>
+<layer number="33" name="tFinish" color="6" fill="3" visible="no" active="no"/>
+<layer number="34" name="bFinish" color="6" fill="6" visible="no" active="no"/>
+<layer number="35" name="tGlue" color="7" fill="4" visible="no" active="no"/>
+<layer number="36" name="bGlue" color="7" fill="5" visible="no" active="no"/>
+<layer number="37" name="tTest" color="7" fill="1" visible="no" active="no"/>
+<layer number="38" name="bTest" color="7" fill="1" visible="no" active="no"/>
+<layer number="39" name="tKeepout" color="4" fill="11" visible="no" active="no"/>
+<layer number="40" name="bKeepout" color="1" fill="11" visible="no" active="no"/>
+<layer number="41" name="tRestrict" color="4" fill="10" visible="no" active="no"/>
+<layer number="42" name="bRestrict" color="1" fill="10" visible="no" active="no"/>
+<layer number="43" name="vRestrict" color="2" fill="10" visible="no" active="no"/>
+<layer number="44" name="Drills" color="7" fill="1" visible="no" active="no"/>
+<layer number="45" name="Holes" color="7" fill="1" visible="no" active="no"/>
+<layer number="46" name="Milling" color="3" fill="1" visible="no" active="no"/>
+<layer number="47" name="Measures" color="7" fill="1" visible="no" active="no"/>
+<layer number="48" name="Document" color="7" fill="1" visible="no" active="no"/>
+<layer number="49" name="Reference" color="7" fill="1" visible="no" active="no"/>
+<layer number="51" name="tDocu" color="7" fill="1" visible="no" active="no"/>
+<layer number="52" name="bDocu" color="7" fill="1" visible="no" active="no"/>
 <layer number="90" name="Modules" color="5" fill="1" visible="yes" active="yes"/>
 <layer number="91" name="Nets" color="2" fill="1" visible="yes" active="yes"/>
@@
 </classes>
 <parts>
+<part name="J_ULTRASONIC_1" library="Ultrasonic Sensor HC-SR04" deviceset="HC-SR04" device=""/>
+<part name="J_ULTRASONIC_2" library="Ultrasonic Sensor HC-SR04" deviceset="HC-SR04" device=""/>
+<part name="J_ULTRASONIC_3" library="Ultrasonic Sensor HC-SR04" deviceset="HC-SR04" device=""/>
+<part name="J_ULTRASONIC_8" library="Ultrasonic Sensor HC-SR04" deviceset="HC-SR04" device=""/>
+<part name="J_ULTRASONIC_5" library="Ultrasonic Sensor HC-SR04" deviceset="HC-SR04" device=""/>
+<part name="J_ULTRASONIC_6" library="Ultrasonic Sensor HC-SR04" deviceset="HC-SR04" device=""/>
+<part name="J_ULTRASONIC_7" library="Ultrasonic Sensor HC-SR04" deviceset="HC-SR04" device=""/>
+<part name="J_ULTRASONIC_4" library="Ultrasonic Sensor HC-SR04" deviceset="HC-SR04" device=""/>
 </parts>
 <sheets>
@@
 </plain>
 <instances>
+<instance part="J_ULTRASONIC_1" gate="J_ULTRASONIC" x="81.28" y="81.28" rot="R90"/>
+<instance part="J_ULTRASONIC_2" gate="J_ULTRASONIC" x="119.38" y="68.58" rot="R90"/>
+<instance part="J_ULTRASONIC_3" gate="J_ULTRASONIC" x="152.4" y="50.8" rot="R90"/>
+<instance part="J_ULTRASONIC_8" gate="J_ULTRASONIC" x="48.26" y="68.58" rot="R90"/>
+<instance part="J_ULTRASONIC_5" gate="J_ULTRASONIC" x="83.82" y="15.24" rot="R90"/>
+<instance part="J_ULTRASONIC_6" gate="J_ULTRASONIC" x="48.26" y="27.94" rot="R90"/>
+<instance part="J_ULTRASONIC_7" gate="J_ULTRASONIC" x="20.32" y="48.26" rot="R90"/>
+<instance part="J_ULTRASONIC_4" gate="J_ULTRASONIC" x="119.38" y="27.94" rot="R90"/>
 </instances>
 <busses>
