File: hardware/eagle/multisonar_shield.brd (EAGLE design)
At the start: 99 x 99 mm, 10 parts, among them J1 ARDUINO_R3_SHIELDUNO_R3_SHIEL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

Commit message: Fixed a few glitches
Routing:
- net SDA: track 65.1 -> 71.9 mm, vias 0 -> 2
- net GND: track 329.9 -> 328.7 mm
- net PC1: track 79.3 -> 78.6 mm
Changed lines of the file:
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@@
 <wire x1="106.5802" y1="64.72" x2="106.8602" y2="65" width="0.6096" layer="16"/>
 <wire x1="58.0662" y1="48.21" x2="58.3202" y2="50.75" width="0.6096" layer="16"/>
-<wire x1="58.0662" y1="48.21" x2="59.0302" y2="47.5" width="0.6096" layer="16"/>
 <wire x1="40" y1="30" x2="40" y2="40" width="0.6096" layer="16"/>
 <wire x1="40" y1="30" x2="45" y2="25" width="0.6096" layer="16"/>
@@
 <wire x1="106.3802" y1="70" x2="106.5802" y2="69.8" width="0.6096" layer="1"/>
 <contactref element="J1" pad="A4"/>
-<wire x1="106.5802" y1="69.8" x2="88.5327" y2="51.7525" width="0.4572" layer="1"/>
-<wire x1="81.915" y1="51.7525" x2="73.9775" y2="43.815" width="0.4572" layer="1"/>
-<wire x1="88.5327" y1="51.7525" x2="81.915" y2="51.7525" width="0.4572" layer="1"/>
-<wire x1="58.0662" y1="30.43" x2="60.0212" y2="32.385" width="0.4572" layer="16"/>
-<wire x1="60.0212" y1="32.385" x2="61.595" y2="32.385" width="0.4572" layer="16"/>
-<wire x1="64.4779" y1="36.44750625" x2="64.83499375" y2="36.8046" width="0.4572" layer="16"/>
-<wire x1="64.83499375" y1="36.8046" x2="65.78749375" y2="36.8046" width="0.4572" layer="16"/>
-<wire x1="61.595" y1="32.385" x2="64.4779" y2="35.2679" width="0.4572" layer="16"/>
-<wire x1="64.4779" y1="35.2679" x2="64.4779" y2="36.44750625" width="0.4572" layer="16"/>
-<wire x1="72.79789375" y1="43.815" x2="73.2536" y2="43.815" width="0.4572" layer="16"/>
-<wire x1="65.78749375" y1="36.8046" x2="72.79789375" y2="43.815" width="0.4572" layer="16"/>
-<wire x1="73.2536" y1="43.815" x2="73.9775" y2="43.815" width="0" layer="19" extent="1-16"/>
+<wire x1="106.5802" y1="69.8" x2="96.4702" y2="59.69" width="0.4064" layer="1"/>
+<wire x1="74.93" y1="46.0375" x2="73.9775" y2="46.0375" width="0.4064" layer="1"/>
+<wire x1="73.9775" y1="46.0375" x2="72.39" y2="44.45" width="0.4064" layer="1"/>
+<wire x1="72.39" y1="44.45" x2="72.39" y2="38.735" width="0.4064" layer="1"/>
+<wire x1="66.3575" y1="32.7025" x2="64.135" y2="32.7025" width="0.4064" layer="1"/>
+<wire x1="64.135" y1="32.7025" x2="63.8175" y2="33.02" width="0.4064" layer="1"/>
+<wire x1="63.8175" y1="33.02" x2="63.8175" y2="35.2425" width="0.4064" layer="1"/>
+<wire x1="96.4702" y1="59.69" x2="88.5825" y2="59.69" width="0.4064" layer="1"/>
+<wire x1="88.5825" y1="59.69" x2="74.93" y2="46.0375" width="0.4064" layer="1"/>
+<wire x1="72.39" y1="38.735" x2="66.3575" y2="32.7025" width="0.4064" layer="1"/>
+<via x="63.8175" y="35.2425" extent="1-16" drill="0.381"/>
+<via x="63.8175" y="35.2425" extent="1-16" drill="0.381"/>
+<wire x1="63.8175" y1="35.2425" x2="59.005" y2="30.43" width="0.4064" layer="16"/>
+<wire x1="59.005" y1="30.43" x2="58.0662" y2="30.43" width="0.4064" layer="16"/>
 </signal>
 <signal name="SCL">
@@
 <via x="64.4525" y="45.72" extent="1-16" drill="0.381"/>
 <wire x1="64.4525" y1="45.72" x2="61.2775" y2="42.545" width="0.4572" layer="16"/>
-<wire x1="61.2775" y1="42.545" x2="60.6425" y2="42.545" width="0.4572" layer="16"/>
 <wire x1="58.3202" y1="38.05" x2="59.0052" y2="38.735" width="0.4572" layer="1"/>
 <wire x1="59.0052" y1="38.735" x2="60.325" y2="38.735" width="0.4572" layer="1"/>
 <wire x1="60.325" y1="38.735" x2="61.0489" y2="39.4589" width="0.4572" layer="1"/>
 <wire x1="61.0489" y1="39.4589" x2="61.0489" y2="42.545" width="0.4572" layer="1"/>
-<wire x1="61.0489" y1="42.545" x2="60.6425" y2="42.545" width="0" layer="19" extent="1-16"/>
+<wire x1="61.0489" y1="42.545" x2="61.2775" y2="42.545" width="0" layer="19" extent="1-16"/>
 </signal>
 <signal name="PC2">
@@
 <via x="60.96" y="42.545" extent="1-16" drill="0.381"/>
 </signal>
-<signal name="N$5">
-<via x="73.9775" y="43.815" extent="1-16" drill="0.381"/>
-</signal>
-<signal name="N$4">
-<via x="108.9025" y="54.2925" extent="1-16" drill="0.381"/>
-</signal>
 </signals>

Commit message: Fixed DRC errors
Routing:
- net SCL: track 70.0 -> 70.8 mm, vias 2 -> 1
- net PC1: track 78.6 -> 79.3 mm, vias 2 -> 3
- net PD3: track 96.4 -> 96.9 mm, vias 4 -> 3
- net PD7: track 72.0 -> 71.5 mm, vias 3 -> 2
- net PB2: track 47.1 -> 46.8 mm, vias 2 -> 1
- net SDA: vias 2 -> 1
Other:
- board text removed: "GND"
- board text removed: "INT"
- board text removed: "RX"
- board text removed: "SCL"
- board text removed: "SDA"
- board text removed: "TX"
